File: sam9x60d5m_basic.kicad_sch (KiCad schematic)
At the start: 34 parts, among them SW1 SW_Push, U1 ME6211C33M5, U2 LR8103B-T18, U3 VRH1202LT, U4 NUC980DR61, U5 AP2127K-ADJ, Y1 12M

Commit message: Finish buck converters; include custom symbols and footprints
Parts:
- removed C1, C11, C22: 10u, symbol Device:C_Small
- removed C10, C13, C14, C15, C16, C17, C18, C19, C20, C21, C3, C4, C5, C6, C7, C8, C9: 100n, symbol Device:C_Small
- removed C12, C2, C23, C26: 1u, symbol Device:C_Small
- removed C24, C25: 15p, symbol Device:C_Small
- removed SW1: SW_Push, symbol Switch:SW_Push
- removed U1: ME6211C33M5, Package_TO_SOT_SMD:SOT-23-5, symbol NUC980:ME6211C33M5
- removed U2: LR8103B-T18, Package_TO_SOT_SMD:SOT-23-5, symbol NUC980:LR8103B
- removed U3: VRH1202LT, Package_TO_SOT_SMD:SOT-23-5, symbol NUC980:VRH1202LT
- removed U4: NUC980DR61, Package_QFP:LQFP-64-1EP_10x10mm_P0.5mm_EP6.5x6.5mm_ThermalVias, symbol CPU_Nuvoton:NUC980DR61
- removed U5: AP2127K-ADJ, Package_TO_SOT_SMD:SOT-23-5, symbol Regulator_Linear:AP2127K-ADJ
- removed Y1: 12M, symbol Device:Crystal_Small
- added J1: Barrel_Jack_Switch, Connector_BarrelJack:BarrelJack_Horizontal, symbol Connector:Barrel_Jack_Switch
- added J2, J3, J4: USB_A, Connector_USB:USB_A_Molex_67643_Horizontal, symbol Connector:USB_A
- added U1: SAM9X60D, SAM9X60D:BGA-233_14x14mm_Layout17x17_P0.8mm_Ball0.4mm, symbol SAM9X60D:SAM9X60D
- R1: value 1M -> 5k62 ±1%; footprint (none) -> Resistor_SMD:R_0603_1608Metric_Pad0.98x0.95mm_HandSolder
Connections:
- net +1V15: now also U1.D6 (VDDCORE), U1.D8 (VDDCORE), U1.G5 (VDDCORE), U1.L6 (VDDCORE), U1.M7 (VDDCORE)
- net +1V8: now also U1.A16 (DDRM_VDD), U1.B15 (DDRM_VDD), U1.B17 (DDRM_VDD), U1.C14 (DDRM_VDD), U1.C16 (DDRM_VDD), U1.D11 (VDDIOM), U1.D13 (DDRM_VDD), U1.D15 (DDRM_VDD), U1.E11 (DDRM_VDD), U1.E12 (DDRM_VDD), U1.E14 (VDDIOM), U1.F13 (DDRM_VDD), U1.G13 (DDRM_VDD), U1.G14 (VDDIOM)
- net +3V3: now also U1.C6 (VDDQSPI), U1.F5 (VDDIOP0), U1.K4 (VDDIOP0), U1.L4 (VDDIOP0), U1.M15 (VDDNF), U1.M3 (VDDIOP1), U1.N11 (VDDIN33), U1.R12 (VDDIN33), U1.R6 (VDDBU)
- net OSC1 renamed USB_RTUNE
- net USB_RTUNE: now also U1.P17 (RTUNE)
- net OSC2 renamed DDRM_VSS
- net DDRM_VSS: now also J1.2, J2.4 (GND), J2.5 (Shield), J3.4 (GND), J3.5 (Shield), J4.4 (GND), J4.5 (Shield), U1.A1 (GND), U1.A13 (GND), U1.A15 (GND), U1.A17 (DDRM_VSS), U1.B13 (GND), U1.B14 (GND), U1.B16 (DDRM_VSS), U1.B2 (GND), U1.C12 (DDRM_VSS), U1.C13 (GND), U1.C15 (DDRM_VSS), U1.C3 (GNDANA), U1.C9 (GND), U1.D14 (DDRM_VSS), U1.D4 (GND), U1.E13 (DDRM_VSS), U1.E5 (GND), U1.E6 (GND), U1.E7 (GND), U1.F11 (DDRM_VSS), U1.F12 (DDRM_VSS), U1.F15 (DDRM_VSS), U1.F3 (GND), U1.F6 (GND), U1.F7 (GND), U1.G12 (DDRM_VSS), U1.G6 (GND), U1.H10 (GND), U1.H8 (GND), U1.H9 (GND), U1.J10 (GND), U1.J15 (GND), U1.J3 (GND), U1.J8 (GND), U1.J9 (GND), U1.K10 (GND), U1.K8 (GND), U1.K9 (GND), U1.L12 (GND), U1.L13 (GND), U1.L14 (GND), U1.L5 (GND), U1.M11 (GND), U1.M12 (GND), U1.M13 (GND), U1.M14 (GND), U1.M5 (GND), U1.M6 (GND), U1.N12 (GND), U1.N13 (GND), U1.N5 (GND), U1.N6 (GND), U1.N7 (GNDIN33), U1.P10 (GND), U1.P14 (GND), U1.P4 (GND), U1.P7 (GNDIN33), U1.R11 (GND), U1.R15 (GND), U1.R16 (GND), U1.R3 (GND), U1.R9 (GND), U1.T16 (GND), U1.T2 (GND), U1.U1 (GND), U1.U15 (GND), U1.U17 (GND)
- new net +3V3A: U1.C2 (VDDANA)
- new net POWER_IN: J1.1
- new net USBA_D+: J2.2 (D-), U1.T15 (HHSDPA)
- new net USBA_D-: J2.3 (D+), U1.U16 (HHSDMA)
- new net USBB_D+: J3.3 (D+), U1.T17 (HHSDPB)
- new net USBB_D-: J3.2 (D-), U1.R17 (HHSDMB)
- new net USBC_D+: J4.3 (D+), U1.P16 (HHSDPC)
- new net USBC_D-: J4.2 (D-), U1.P15 (HHSDMC)
- no-connect marks 0 -> 1
Other:
- added sheet Power (sam9x60d5m_basic_power.kicad_sch)
- title: (none) -> SAM9X60D Basic Eval Board
